Commit message: Se añadio el archivo gazebo.launch.py para lanzar gazebo, se hicieron unos cambios en package.xml y se añadieron las notas de clase 44

File: arduinobot_ws/install/arduinobot_description/share/arduinobot_description/urdf/arduinobot.urdf.xacro (robot description, xacro)
@@ -6,12 +6,29 @@
   <xacro:property name="path" value="package://arduinobot_description/meshes/" />
   <xacro:property name="scale" value="0.01 0.01 0.01"/>
+  <xacro:macro name="default_inertial" params="mass">
+    <inertial>
+      <mass value="${mass}" />
+      <inertia
+        ixx="1.0" ixy="0.0" ixz="0.0"
+        iyy="1.0" iyz="0.0"
+        izz="1.0"
+      />
+    </inertial>
+  </xacro:macro>
   <link name="world"/>
   <link name="base_link">
+    <xacro:default_inertial mass="1.0" />
     <visual>
       <origin xyz="-0.5 -0.5 0" rpy="0 0 0"/>
       <geometry>
-        <mesh filename="package://arduinobot_description/meshes/basement.STL" scale="0.01 0.01 0.01"/>
+        <mesh filename="${path}basement.STL" scale="0.01 0.01 0.01"/>
       </geometry>
     </visual>
+    <collision>
+      <origin xyz="-0.5 -0.5 0" rpy="0 0 0"/>
+      <geometry>
+        <mesh filename="${path}basement.STL" scale="0.01 0.01 0.01"/>
+      </geometry>
+    </collision>
   </link>
   <joint name="virtual_joint" type="fixed">
@@ -21,10 +38,17 @@
   </joint>
   <link name="base_plate">
+    <xacro:default_inertial mass="0.1" />
     <visual>
       <origin rpy="0 0 0" xyz="-0.39 -0.39 -0.56"/>
       <geometry>
-        <mesh filename="package://arduinobot_description/meshes/base_plate.STL" scale="0.01 0.01 0.01"/>
+        <mesh filename="${path}base_plate.STL" scale="0.01 0.01 0.01"/>
       </geometry>
     </visual>
+    <collision>
+      <origin rpy="0 0 0" xyz="-0.39 -0.39 -0.56"/>
+      <geometry>
+        <mesh filename="${path}base_plate.STL" scale="0.01 0.01 0.01"/>
+      </geometry>
+    </collision>
   </link>
   <joint name="joint_1" type="revolute">
@@ -36,4 +60,5 @@
   </joint>
   <link name="forward_drive_arm">
+    <xacro:default_inertial mass="0.1" />
     <visual>
       <origin xyz="0.19 0.06 -0.08" rpy="0 -${PI/2} ${PI/2}" />
@@ -42,4 +67,10 @@
       </geometry>
     </visual>
+    <collision>
+      <origin xyz="0.19 0.06 -0.08" rpy="0 -${PI/2} ${PI/2}" />
+      <geometry>
+        <mesh filename="${path}forward_drive_arm.STL" scale="${scale}"/>
+      </geometry>
+    </collision>
   </link>
   <joint name="joint_2" type="revolute">
@@ -51,4 +82,5 @@
   </joint>
   <link name="horizontal_arm">
+    <xacro:default_inertial mass="0.1" />
     <visual>
       <origin xyz="-0.03 -0.4 -0.06" rpy="${PI/2} 0 ${PI/2}" />
@@ -60,4 +92,13 @@
       </material>
     </visual>
+    <collision>
+      <origin xyz="-0.03 -0.4 -0.06" rpy="${PI/2} 0 ${PI/2}" />
+      <geometry>
+        <mesh filename="${path}horizontal_arm.STL" scale="${scale}"/>
+      </geometry>
+      <material name="material_name">
+        <color rgba="1 1 1 1" />
+      </material>
+    </collision>
   </link>
   <joint name="joint_3" type="revolute">
@@ -69,4 +110,5 @@
   </joint>
   <link name="claw_support">
+    <xacro:default_inertial mass="0.05" />
     <visual>
       <origin xyz="0 -0.05 -0.15" rpy="0 0 ${PI/2}"/>
@@ -75,4 +117,10 @@
       </geometry>
     </visual>
+    <collision>
+      <origin xyz="0 -0.05 -0.15" rpy="0 0 ${PI/2}"/>
+      <geometry>
+        <mesh filename="${path}claw_support.STL" scale="${scale}"/>
+      </geometry>
+    </collision>
   </link>
   <joint name="horizontal_arm_to_claw_support" type="fixed">
@@ -82,4 +130,5 @@
   </joint>
   <link name="gripper_right">
+    <xacro:default_inertial mass="0.01" />
     <visual>
       <origin xyz="-0.1 0.5 -0.1" rpy="0 0 -${PI/2}" />
@@ -88,6 +137,13 @@
       </geometry>
     </visual>
+    <collision>
+      <origin xyz="-0.1 0.5 -0.1" rpy="0 0 -${PI/2}" />
+      <geometry>
+        <mesh filename="${path}right_finger.STL" scale="${scale}"/>
+      </geometry>
+    </collision>
   </link>
   <link name="gripper_left">
+    <xacro:default_inertial mass="0.01" />
     <visual>
       <origin xyz="-0.04 0.5 -0.1" rpy="0 0 -${PI/2}" />
@@ -96,4 +152,10 @@
       </geometry>
     </visual>
+    <collision>
+      <origin xyz="-0.04 0.5 -0.1" rpy="0 0 -${PI/2}" />
+      <geometry>
+        <mesh filename="${path}left_finger.STL" scale="${scale}"/>
+      </geometry>
+    </collision>
   </link>
   <joint name="joint_4" type="revolute">
@@ -112,3 +174,22 @@
     <limit lower="0.0" upper="${PI/2}" effort="${effort}" velocity="${velocity}" />
   </joint>
+  <link name="rgb_camera">
+      <visual>
+          <origin rpy="-1.57 0 -1.57" xyz="-0.1 0.125 0.15"/>
+          <geometry>
+              <mesh filename="${path}pi_camera.STL" scale="${scale}"/>
+          </geometry>
+      </visual>
+      <collision>
+        <origin rpy="-1.57 0 -1.57" xyz="-0.1 0.125 0.15"/>
+        <geometry>
+            <mesh filename="${path}pi_camera.STL" scale="${scale}"/>
+        </geometry>
+      </collision>
+  </link>
+  <joint name ="rgb_camera_joint" type="fixed">
+      <parent link="base_link"/>
+      <child link = "rgb_camera"/>
+      <origin xyz="0 0.45 0.2" rpy="0 -0.5 1.57"/>
+  </joint>
 </robot>
