Commit message: se hizo la clase 33 con sus notas

File: arduinobot_ws/src/arduinobot_description/urdf/arduinobot.urdf.xacro (robot description, xacro)
@@ -4,4 +4,6 @@
   <xacro:property name="effort" value="30.0"/>
   <xacro:property name="velocity" value="10.0"/>
+  <xacro:property name="path" value="package://arduinobot_description/meshes/" />
+  <xacro:property name="scale" value="0.01 0.01 0.01"/>
   <link name="world"/>
   <link name="base_link">
@@ -33,3 +35,80 @@
     <limit lower="-${PI / 2}" upper="${PI / 2}" effort="${effort}" velocity="${velocity}"/>
   </joint>
+  <link name="forward_drive_arm">
+    <visual>
+      <origin xyz="0.19 0.06 -0.08" rpy="0 -${PI/2} ${PI/2}" />
+      <geometry>
+        <mesh filename="${path}forward_drive_arm.STL" scale="${scale}"/>
+      </geometry>
+    </visual>
+  </link>
+  <joint name="joint_2" type="revolute">
+    <parent link="base_plate" />
+    <child link="forward_drive_arm" />
+    <origin xyz="-0.02 0 0.35" rpy="0 0 0"/>
+    <axis xyz="1 0 0" />
+    <limit lower="-${PI/2}" upper="${PI/2}" effort="${effort}" velocity="${velocity}" />
+  </joint>
+  <link name="horizontal_arm">
+    <visual>
+      <origin xyz="-0.03 -0.4 -0.06" rpy="${PI/2} 0 ${PI/2}" />
+      <geometry>
+        <mesh filename="${path}horizontal_arm.STL" scale="${scale}"/>
+      </geometry>
+      <material name="material_name">
+        <color rgba="1 1 1 1" />
+      </material>
+    </visual>
+  </link>
+  <joint name="joint_3" type="revolute">
+    <parent link="forward_drive_arm" />
+    <child link="horizontal_arm" />
+    <axis xyz="1 0 0" />
+    <origin rpy="0 0 0" xyz="0 0 0.8" />
+    <limit lower="-${PI/2}" upper="${PI/2}" effort="${effort}" velocity="${velocity}" />
+  </joint>
+  <link name="claw_support">
+    <visual>
+      <origin xyz="0 -0.05 -0.15" rpy="0 0 ${PI/2}"/>
+      <geometry>
+        <mesh filename="${path}claw_support.STL" scale="${scale}"/>
+      </geometry>
+    </visual>
+  </link>
+  <joint name="horizontal_arm_to_claw_support" type="fixed">
+    <parent link="horizontal_arm" />
+    <child link="claw_support" />
+    <origin xyz="0 0.82 0" rpy="0 0 0" />
+  </joint>
+  <link name="gripper_right">
+    <visual>
+      <origin xyz="-0.1 0.5 -0.1" rpy="0 0 -${PI/2}" />
+      <geometry>
+        <mesh filename="${path}right_finger.STL" scale="${scale}"/>
+      </geometry>
+    </visual>
+  </link>
+  <link name="gripper_left">
+    <visual>
+      <origin xyz="-0.04 0.5 -0.1" rpy="0 0 -${PI/2}" />
+      <geometry>
+        <mesh filename="${path}left_finger.STL" scale="${scale}"/>
+      </geometry>
+    </visual>
+  </link>
+  <joint name="joint_4" type="revolute">
+    <parent link="claw_support" />
+    <child link="gripper_right" />
+    <origin xyz="-0.04 0.13 -0.1" rpy="0 0 0" />
+    <axis xyz="0 0 1" />
+    <limit lower="-${PI/2}" upper="0.0" effort="${effort}" velocity="${velocity}" />
+  </joint>
+  <joint name="joint_5" type="revolute">
+    <parent link="claw_support" />
+    <child link="gripper_left" />
+    <origin xyz="-0.22 0.13 -0.1" rpy="0 0 0" />
+    <axis xyz="0 0 1" />
+    <mimic joint="joint_4" multiplier="-1"/>
+    <limit lower="0.0" upper="${PI/2}" effort="${effort}" velocity="${velocity}" />
+  </joint>
 </robot>

Commit message: Se añadio una camara RGB a URDF, se añadieron las notas de clase 42

File: arduinobot_ws/src/arduinobot_description/urdf/arduinobot.urdf.xacro (robot description, xacro)
@@ -11,5 +11,5 @@
       <origin xyz="-0.5 -0.5 0" rpy="0 0 0"/>
       <geometry>
-        <mesh filename="package://arduinobot_description/meshes/basement.STL" scale="0.01 0.01 0.01"/>
+        <mesh filename="${path}basement.STL" scale="0.01 0.01 0.01"/>
       </geometry>
     </visual>
@@ -24,5 +24,5 @@
       <origin rpy="0 0 0" xyz="-0.39 -0.39 -0.56"/>
       <geometry>
-        <mesh filename="package://arduinobot_description/meshes/base_plate.STL" scale="0.01 0.01 0.01"/>
+        <mesh filename="${path}base_plate.STL" scale="0.01 0.01 0.01"/>
       </geometry>
     </visual>
@@ -112,3 +112,16 @@
     <limit lower="0.0" upper="${PI/2}" effort="${effort}" velocity="${velocity}" />
   </joint>
+  <link name="rgb_camera">
+      <visual>
+          <origin rpy="-1.57 0 -1.57" xyz="-0.1 0.125 0.15"/>
+          <geometry>
+              <mesh filename="${path}pi_camera.STL" scale="${scale}"/>
+          </geometry>
+      </visual>
+  </link>
+  <joint name ="rgb_camera_joint" type="fixed">
+      <parent link="base_link"/>
+      <child link = "rgb_camera"/>
+      <origin xyz="0 0.45 0.2" rpy="0 -0.5 1.57"/>
+  </joint>
 </robot>

Commit message: se añadieron notas de clas 43

File: arduinobot_ws/src/arduinobot_description/urdf/arduinobot.urdf.xacro (robot description, xacro)
@@ -6,6 +6,17 @@
   <xacro:property name="path" value="package://arduinobot_description/meshes/" />
   <xacro:property name="scale" value="0.01 0.01 0.01"/>
+  <xacro:macro name="default_inertial" params="mass">
+    <inertial>
+      <mass value="${mass}" />
+      <inertia
+        ixx="1.0" ixy="0.0" ixz="0.0"
+        iyy="1.0" iyz="0.0"
+        izz="1.0"
+      />
+    </inertial>
+  </xacro:macro>
   <link name="world"/>
   <link name="base_link">
+    <xacro:default_inertial mass="1.0" />
     <visual>
       <origin xyz="-0.5 -0.5 0" rpy="0 0 0"/>
@@ -14,4 +25,10 @@
       </geometry>
     </visual>
+    <collision>
+      <origin xyz="-0.5 -0.5 0" rpy="0 0 0"/>
+      <geometry>
+        <mesh filename="${path}basement.STL" scale="0.01 0.01 0.01"/>
+      </geometry>
+    </collision>
   </link>
   <joint name="virtual_joint" type="fixed">
@@ -21,4 +38,5 @@
   </joint>
   <link name="base_plate">
+    <xacro:default_inertial mass="0.1" />
     <visual>
       <origin rpy="0 0 0" xyz="-0.39 -0.39 -0.56"/>
@@ -27,4 +45,10 @@
       </geometry>
     </visual>
+    <collision>
+      <origin rpy="0 0 0" xyz="-0.39 -0.39 -0.56"/>
+      <geometry>
+        <mesh filename="${path}base_plate.STL" scale="0.01 0.01 0.01"/>
+      </geometry>
+    </collision>
   </link>
   <joint name="joint_1" type="revolute">
@@ -36,4 +60,5 @@
   </joint>
   <link name="forward_drive_arm">
+    <xacro:default_inertial mass="0.1" />
     <visual>
       <origin xyz="0.19 0.06 -0.08" rpy="0 -${PI/2} ${PI/2}" />
@@ -42,4 +67,10 @@
       </geometry>
     </visual>
+    <collision>
+      <origin xyz="0.19 0.06 -0.08" rpy="0 -${PI/2} ${PI/2}" />
+      <geometry>
+        <mesh filename="${path}forward_drive_arm.STL" scale="${scale}"/>
+      </geometry>
+    </collision>
   </link>
   <joint name="joint_2" type="revolute">
@@ -51,4 +82,5 @@
   </joint>
   <link name="horizontal_arm">
+    <xacro:default_inertial mass="0.1" />
     <visual>
       <origin xyz="-0.03 -0.4 -0.06" rpy="${PI/2} 0 ${PI/2}" />
@@ -60,4 +92,13 @@
       </material>
     </visual>
+    <collision>
+      <origin xyz="-0.03 -0.4 -0.06" rpy="${PI/2} 0 ${PI/2}" />
+      <geometry>
+        <mesh filename="${path}horizontal_arm.STL" scale="${scale}"/>
+      </geometry>
+      <material name="material_name">
+        <color rgba="1 1 1 1" />
+      </material>
+    </collision>
   </link>
   <joint name="joint_3" type="revolute">
@@ -69,4 +110,5 @@
   </joint>
   <link name="claw_support">
+    <xacro:default_inertial mass="0.05" />
     <visual>
       <origin xyz="0 -0.05 -0.15" rpy="0 0 ${PI/2}"/>
@@ -75,4 +117,10 @@
       </geometry>
     </visual>
+    <collision>
+      <origin xyz="0 -0.05 -0.15" rpy="0 0 ${PI/2}"/>
+      <geometry>
+        <mesh filename="${path}claw_support.STL" scale="${scale}"/>
+      </geometry>
+    </collision>
   </link>
   <joint name="horizontal_arm_to_claw_support" type="fixed">
@@ -82,4 +130,5 @@
   </joint>
   <link name="gripper_right">
+    <xacro:default_inertial mass="0.01" />
     <visual>
       <origin xyz="-0.1 0.5 -0.1" rpy="0 0 -${PI/2}" />
@@ -88,6 +137,13 @@
       </geometry>
     </visual>
+    <collision>
+      <origin xyz="-0.1 0.5 -0.1" rpy="0 0 -${PI/2}" />
+      <geometry>
+        <mesh filename="${path}right_finger.STL" scale="${scale}"/>
+      </geometry>
+    </collision>
   </link>
   <link name="gripper_left">
+    <xacro:default_inertial mass="0.01" />
     <visual>
       <origin xyz="-0.04 0.5 -0.1" rpy="0 0 -${PI/2}" />
@@ -96,4 +152,10 @@
       </geometry>
     </visual>
+    <collision>
+      <origin xyz="-0.04 0.5 -0.1" rpy="0 0 -${PI/2}" />
+      <geometry>
+        <mesh filename="${path}left_finger.STL" scale="${scale}"/>
+      </geometry>
+    </collision>
   </link>
   <joint name="joint_4" type="revolute">
@@ -119,4 +181,10 @@
           </geometry>
       </visual>
+      <collision>
+        <origin rpy="-1.57 0 -1.57" xyz="-0.1 0.125 0.15"/>
+        <geometry>
+            <mesh filename="${path}pi_camera.STL" scale="${scale}"/>
+        </geometry>
+      </collision>
   </link>
   <joint name ="rgb_camera_joint" type="fixed">
