Commit message: se añadieron las modificaciones a la tarea de clase 44

File: arduinobot_ws/src/arduinobot_description/urdf/arduinobot.urdf.xacro (robot description, xacro)
@@ -1,12 +1,22 @@
 <?xml version="1.0"?>
+<!-- Declaración XML estándar del documento. -->
 <robot xmlns:xacro="http://www.ros.org/wiki/xacro" name="arduinobot">
+<!-- Elemento raíz URDF; define el nombre del robot y el espacio de nombres de Xacro. -->
   <xacro:property name="PI" value="3.14159" />
+  <!-- Propiedad Xacro: constante PI para cálculos en radianes. -->
   <xacro:property name="effort" value="30.0"/>
+  <!-- Propiedad Xacro: esfuerzo máximo por defecto de juntas (p. ej., N·m). -->
   <xacro:property name="velocity" value="10.0"/>
+  <!-- Propiedad Xacro: velocidad máxima por defecto de juntas (rad/s). -->
   <xacro:property name="path" value="package://arduinobot_description/meshes/" />
+  <!-- Propiedad Xacro: ruta base a las mallas del robot (package://...). -->
   <xacro:property name="scale" value="0.01 0.01 0.01"/>
+  <!-- Propiedad Xacro: factor de escala aplicado a las mallas importadas. -->
   <xacro:macro name="default_inertial" params="mass">
+  <!-- Declaración de la macro Xacro 'default_inertial' para insertar bloques <inertial> reutilizables. -->
     <inertial>
+    <!-- Inicio del bloque inercial: define masa y tensor de inercia del enlace. -->
       <mass value="${mass}" />
+      <!-- Masa del enlace (en kilogramos). -->
       <inertia
         ixx="1.0" ixy="0.0" ixz="0.0"
@@ -15,196 +25,381 @@
       />
     </inertial>
+      <!-- Tensor de inercia (ixx, iyy, izz, etc.) respecto al centro de masa. -->
+    <!-- Fin del bloque inercial. -->
   </xacro:macro>
   <link name="world"/>
+  <!-- Definición de un enlace rígido del robot: 'world'. -->
   <link name="base_link">
+  <!-- Definición de un enlace rígido del robot: 'base_link'. -->
     <xacro:default_inertial mass="1.0" />
     <visual>
+    <!-- Bloque 'visual': cómo se renderiza el enlace en pantalla. -->
       <origin xyz="-0.5 -0.5 0" rpy="0 0 0"/>
-      <geometry>
+      <!-- Transformación del elemento: posición (xyz en m) y orientación (rpy en rad) respecto al marco padre. -->
+      <geometry>
+      <!-- Inicio de la geometría asociada (malla o primitivas). -->
         <mesh filename="${path}basement.STL" scale="0.01 0.01 0.01"/>
-      </geometry>
-    </visual>
-    <collision>
+        <!-- Carga una malla (STL) desde el paquete; 'scale' ajusta sus dimensiones. -->
+      </geometry>
+      <!-- Fin de la geometría. -->
+    </visual>
+    <!-- Fin del bloque 'visual'. -->
+    <collision>
+    <!-- Bloque 'collision': geometría usada por el motor físico para detección de colisiones. -->
       <origin xyz="-0.5 -0.5 0" rpy="0 0 0"/>
-      <geometry>
+      <!-- Transformación del elemento: posición (xyz en m) y orientación (rpy en rad) respecto al marco padre. -->
+      <geometry>
+      <!-- Inicio de la geometría asociada (malla o primitivas). -->
         <mesh filename="${path}basement.STL" scale="0.01 0.01 0.01"/>
-      </geometry>
-    </collision>
-  </link>
+        <!-- Carga una malla (STL) desde el paquete; 'scale' ajusta sus dimensiones. -->
+      </geometry>
+      <!-- Fin de la geometría. -->
+    </collision>
+    <!-- Fin del bloque 'collision'. -->
+  </link>
+  <!-- Fin de la definición del enlace. -->
   <joint name="virtual_joint" type="fixed">
+  <!-- Articulación 'virtual_joint' de tipo 'fixed' que conecta dos enlaces. -->
     <parent link="world"/>
+    <!-- Especifica el enlace padre conectado por esta articulación. -->
     <child link="base_link"/>
+    <!-- Especifica el enlace hijo conectado por esta articulación. -->
     <origin xyz="0 0 0" rpy="0 0 0"/>
-  </joint>
+    <!-- Transformación del elemento: posición (xyz en m) y orientación (rpy en rad) respecto al marco padre. -->
+  </joint>
+  <!-- Fin de la articulación. -->
   <link name="base_plate">
+  <!-- Definición de un enlace rígido del robot: 'base_plate'. -->
     <xacro:default_inertial mass="0.1" />
     <visual>
+    <!-- Bloque 'visual': cómo se renderiza el enlace en pantalla. -->
       <origin rpy="0 0 0" xyz="-0.39 -0.39 -0.56"/>
-      <geometry>
+      <!-- Transformación del elemento: posición (xyz en m) y orientación (rpy en rad) respecto al marco padre. -->
+      <geometry>
+      <!-- Inicio de la geometría asociada (malla o primitivas). -->
         <mesh filename="${path}base_plate.STL" scale="0.01 0.01 0.01"/>
-      </geometry>
-    </visual>
-    <collision>
+        <!-- Carga una malla (STL) desde el paquete; 'scale' ajusta sus dimensiones. -->
+      </geometry>
+      <!-- Fin de la geometría. -->
+    </visual>
+    <!-- Fin del bloque 'visual'. -->
+    <collision>
+    <!-- Bloque 'collision': geometría usada por el motor físico para detección de colisiones. -->
       <origin rpy="0 0 0" xyz="-0.39 -0.39 -0.56"/>
-      <geometry>
+      <!-- Transformación del elemento: posición (xyz en m) y orientación (rpy en rad) respecto al marco padre. -->
+      <geometry>
+      <!-- Inicio de la geometría asociada (malla o primitivas). -->
         <mesh filename="${path}base_plate.STL" scale="0.01 0.01 0.01"/>
-      </geometry>
-    </collision>
-  </link>
+        <!-- Carga una malla (STL) desde el paquete; 'scale' ajusta sus dimensiones. -->
+      </geometry>
+      <!-- Fin de la geometría. -->
+    </collision>
+    <!-- Fin del bloque 'collision'. -->
+  </link>
+  <!-- Fin de la definición del enlace. -->
   <joint name="joint_1" type="revolute">
+  <!-- Articulación 'joint_1' de tipo 'revolute' que conecta dos enlaces. -->
     <parent link="base_link" />
+    <!-- Especifica el enlace padre conectado por esta articulación. -->
     <child link="base_plate" />
+    <!-- Especifica el enlace hijo conectado por esta articulación. -->
     <origin xyz="0 0 0.307"/>
+    <!-- Transformación del elemento: posición (xyz en m) y orientación (rpy en rad) respecto al marco padre. -->
     <axis xyz="0 0 1" />
+    <!-- Eje de movimiento de la articulación (vector unitario). -->
     <limit lower="-${PI / 2}" upper="${PI / 2}" effort="${effort}" velocity="${velocity}"/>
-  </joint>
+    <!-- Límites de la articulación: rango, esfuerzo y velocidad máximos. -->
+  </joint>
+  <!-- Fin de la articulación. -->
   <link name="forward_drive_arm">
+  <!-- Definición de un enlace rígido del robot: 'forward_drive_arm'. -->
     <xacro:default_inertial mass="0.1" />
     <visual>
+    <!-- Bloque 'visual': cómo se renderiza el enlace en pantalla. -->
       <origin xyz="0.19 0.06 -0.08" rpy="0 -${PI/2} ${PI/2}" />
-      <geometry>
+      <!-- Transformación del elemento: posición (xyz en m) y orientación (rpy en rad) respecto al marco padre. -->
+      <geometry>
+      <!-- Inicio de la geometría asociada (malla o primitivas). -->
         <mesh filename="${path}forward_drive_arm.STL" scale="${scale}"/>
-      </geometry>
-    </visual>
-    <collision>
+        <!-- Carga una malla (STL) desde el paquete; 'scale' ajusta sus dimensiones. -->
+      </geometry>
+      <!-- Fin de la geometría. -->
+    </visual>
+    <!-- Fin del bloque 'visual'. -->
+    <collision>
+    <!-- Bloque 'collision': geometría usada por el motor físico para detección de colisiones. -->
       <origin xyz="0.19 0.06 -0.08" rpy="0 -${PI/2} ${PI/2}" />
-      <geometry>
+      <!-- Transformación del elemento: posición (xyz en m) y orientación (rpy en rad) respecto al marco padre. -->
+      <geometry>
+      <!-- Inicio de la geometría asociada (malla o primitivas). -->
         <mesh filename="${path}forward_drive_arm.STL" scale="${scale}"/>
-      </geometry>
-    </collision>
-  </link>
+        <!-- Carga una malla (STL) desde el paquete; 'scale' ajusta sus dimensiones. -->
+      </geometry>
+      <!-- Fin de la geometría. -->
+    </collision>
+    <!-- Fin del bloque 'collision'. -->
+  </link>
+  <!-- Fin de la definición del enlace. -->
   <joint name="joint_2" type="revolute">
+  <!-- Articulación 'joint_2' de tipo 'revolute' que conecta dos enlaces. -->
     <parent link="base_plate" />
+    <!-- Especifica el enlace padre conectado por esta articulación. -->
     <child link="forward_drive_arm" />
+    <!-- Especifica el enlace hijo conectado por esta articulación. -->
     <origin xyz="-0.02 0 0.35" rpy="0 0 0"/>
+    <!-- Transformación del elemento: posición (xyz en m) y orientación (rpy en rad) respecto al marco padre. -->
     <axis xyz="1 0 0" />
+    <!-- Eje de movimiento de la articulación (vector unitario). -->
     <limit lower="-${PI/2}" upper="${PI/2}" effort="${effort}" velocity="${velocity}" />
-  </joint>
+    <!-- Límites de la articulación: rango, esfuerzo y velocidad máximos. -->
+  </joint>
+  <!-- Fin de la articulación. -->
   <link name="horizontal_arm">
+  <!-- Definición de un enlace rígido del robot: 'horizontal_arm'. -->
     <xacro:default_inertial mass="0.1" />
     <visual>
+    <!-- Bloque 'visual': cómo se renderiza el enlace en pantalla. -->
       <origin xyz="-0.03 -0.4 -0.06" rpy="${PI/2} 0 ${PI/2}" />
-      <geometry>
+      <!-- Transformación del elemento: posición (xyz en m) y orientación (rpy en rad) respecto al marco padre. -->
+      <geometry>
+      <!-- Inicio de la geometría asociada (malla o primitivas). -->
         <mesh filename="${path}horizontal_arm.STL" scale="${scale}"/>
-      </geometry>
+        <!-- Carga una malla (STL) desde el paquete; 'scale' ajusta sus dimensiones. -->
+      </geometry>
+      <!-- Fin de la geometría. -->
       <material name="material_name">
+      <!-- Definición de un material (nombre) para colorear/estilizar visualmente. -->
         <color rgba="1 1 1 1" />
+        <!-- Color RGBA asociado al material (valores entre 0 y 1). -->
       </material>
-    </visual>
-    <collision>
+      <!-- Fin de la definición del material. -->
+    </visual>
+    <!-- Fin del bloque 'visual'. -->
+    <collision>
+    <!-- Bloque 'collision': geometría usada por el motor físico para detección de colisiones. -->
       <origin xyz="-0.03 -0.4 -0.06" rpy="${PI/2} 0 ${PI/2}" />
-      <geometry>
+      <!-- Transformación del elemento: posición (xyz en m) y orientación (rpy en rad) respecto al marco padre. -->
+      <geometry>
+      <!-- Inicio de la geometría asociada (malla o primitivas). -->
         <mesh filename="${path}horizontal_arm.STL" scale="${scale}"/>
-      </geometry>
+        <!-- Carga una malla (STL) desde el paquete; 'scale' ajusta sus dimensiones. -->
+      </geometry>
+      <!-- Fin de la geometría. -->
       <material name="material_name">
+      <!-- Definición de un material (nombre) para colorear/estilizar visualmente. -->
         <color rgba="1 1 1 1" />
+        <!-- Color RGBA asociado al material (valores entre 0 y 1). -->
       </material>
-    </collision>
-  </link>
+      <!-- Fin de la definición del material. -->
+    </collision>
+    <!-- Fin del bloque 'collision'. -->
+  </link>
+  <!-- Fin de la definición del enlace. -->
   <joint name="joint_3" type="revolute">
+  <!-- Articulación 'joint_3' de tipo 'revolute' que conecta dos enlaces. -->
     <parent link="forward_drive_arm" />
+    <!-- Especifica el enlace padre conectado por esta articulación. -->
     <child link="horizontal_arm" />
+    <!-- Especifica el enlace hijo conectado por esta articulación. -->
     <axis xyz="1 0 0" />
+    <!-- Eje de movimiento de la articulación (vector unitario). -->
     <origin rpy="0 0 0" xyz="0 0 0.8" />
+    <!-- Transformación del elemento: posición (xyz en m) y orientación (rpy en rad) respecto al marco padre. -->
     <limit lower="-${PI/2}" upper="${PI/2}" effort="${effort}" velocity="${velocity}" />
-  </joint>
+    <!-- Límites de la articulación: rango, esfuerzo y velocidad máximos. -->
+  </joint>
+  <!-- Fin de la articulación. -->
   <link name="claw_support">
+  <!-- Definición de un enlace rígido del robot: 'claw_support'. -->
     <xacro:default_inertial mass="0.05" />
     <visual>
+    <!-- Bloque 'visual': cómo se renderiza el enlace en pantalla. -->
       <origin xyz="0 -0.05 -0.15" rpy="0 0 ${PI/2}"/>
-      <geometry>
+      <!-- Transformación del elemento: posición (xyz en m) y orientación (rpy en rad) respecto al marco padre. -->
+      <geometry>
+      <!-- Inicio de la geometría asociada (malla o primitivas). -->
         <mesh filename="${path}claw_support.STL" scale="${scale}"/>
-      </geometry>
-    </visual>
-    <collision>
+        <!-- Carga una malla (STL) desde el paquete; 'scale' ajusta sus dimensiones. -->
+      </geometry>
+      <!-- Fin de la geometría. -->
+    </visual>
+    <!-- Fin del bloque 'visual'. -->
+    <collision>
+    <!-- Bloque 'collision': geometría usada por el motor físico para detección de colisiones. -->
       <origin xyz="0 -0.05 -0.15" rpy="0 0 ${PI/2}"/>
-      <geometry>
+      <!-- Transformación del elemento: posición (xyz en m) y orientación (rpy en rad) respecto al marco padre. -->
+      <geometry>
+      <!-- Inicio de la geometría asociada (malla o primitivas). -->
         <mesh filename="${path}claw_support.STL" scale="${scale}"/>
-      </geometry>
-    </collision>
-  </link>
+        <!-- Carga una malla (STL) desde el paquete; 'scale' ajusta sus dimensiones. -->
+      </geometry>
+      <!-- Fin de la geometría. -->
+    </collision>
+    <!-- Fin del bloque 'collision'. -->
+  </link>
+  <!-- Fin de la definición del enlace. -->
   <joint name="horizontal_arm_to_claw_support" type="fixed">
+  <!-- Articulación 'horizontal_arm_to_claw_support' de tipo 'fixed' que conecta dos enlaces. -->
     <parent link="horizontal_arm" />
+    <!-- Especifica el enlace padre conectado por esta articulación. -->
     <child link="claw_support" />
+    <!-- Especifica el enlace hijo conectado por esta articulación. -->
     <origin xyz="0 0.82 0" rpy="0 0 0" />
-  </joint>
+    <!-- Transformación del elemento: posición (xyz en m) y orientación (rpy en rad) respecto al marco padre. -->
+  </joint>
+  <!-- Fin de la articulación. -->
   <link name="gripper_right">
+  <!-- Definición de un enlace rígido del robot: 'gripper_right'. -->
     <xacro:default_inertial mass="0.01" />
     <visual>
+    <!-- Bloque 'visual': cómo se renderiza el enlace en pantalla. -->
       <origin xyz="-0.1 0.5 -0.1" rpy="0 0 -${PI/2}" />
-      <geometry>
+      <!-- Transformación del elemento: posición (xyz en m) y orientación (rpy en rad) respecto al marco padre. -->
+      <geometry>
+      <!-- Inicio de la geometría asociada (malla o primitivas). -->
         <mesh filename="${path}right_finger.STL" scale="${scale}"/>
-      </geometry>
-    </visual>
-    <collision>
+        <!-- Carga una malla (STL) desde el paquete; 'scale' ajusta sus dimensiones. -->
+      </geometry>
+      <!-- Fin de la geometría. -->
+    </visual>
+    <!-- Fin del bloque 'visual'. -->
+    <collision>
+    <!-- Bloque 'collision': geometría usada por el motor físico para detección de colisiones. -->
       <origin xyz="-0.1 0.5 -0.1" rpy="0 0 -${PI/2}" />
-      <geometry>
+      <!-- Transformación del elemento: posición (xyz en m) y orientación (rpy en rad) respecto al marco padre. -->
+      <geometry>
+      <!-- Inicio de la geometría asociada (malla o primitivas). -->
         <mesh filename="${path}right_finger.STL" scale="${scale}"/>
-      </geometry>
-    </collision>
-  </link>
+        <!-- Carga una malla (STL) desde el paquete; 'scale' ajusta sus dimensiones. -->
+      </geometry>
+      <!-- Fin de la geometría. -->
+    </collision>
+    <!-- Fin del bloque 'collision'. -->
+  </link>
+  <!-- Fin de la definición del enlace. -->
   <link name="gripper_left">
+  <!-- Definición de un enlace rígido del robot: 'gripper_left'. -->
     <xacro:default_inertial mass="0.01" />
     <visual>
+    <!-- Bloque 'visual': cómo se renderiza el enlace en pantalla. -->
       <origin xyz="-0.04 0.5 -0.1" rpy="0 0 -${PI/2}" />
-      <geometry>
+      <!-- Transformación del elemento: posición (xyz en m) y orientación (rpy en rad) respecto al marco padre. -->
+      <geometry>
+      <!-- Inicio de la geometría asociada (malla o primitivas). -->
         <mesh filename="${path}left_finger.STL" scale="${scale}"/>
-      </geometry>
-    </visual>
-    <collision>
+        <!-- Carga una malla (STL) desde el paquete; 'scale' ajusta sus dimensiones. -->
+      </geometry>
+      <!-- Fin de la geometría. -->
+    </visual>
+    <!-- Fin del bloque 'visual'. -->
+    <collision>
+    <!-- Bloque 'collision': geometría usada por el motor físico para detección de colisiones. -->
       <origin xyz="-0.04 0.5 -0.1" rpy="0 0 -${PI/2}" />
-      <geometry>
+      <!-- Transformación del elemento: posición (xyz en m) y orientación (rpy en rad) respecto al marco padre. -->
+      <geometry>
+      <!-- Inicio de la geometría asociada (malla o primitivas). -->
         <mesh filename="${path}left_finger.STL" scale="${scale}"/>
-      </geometry>
-    </collision>
-  </link>
+        <!-- Carga una malla (STL) desde el paquete; 'scale' ajusta sus dimensiones. -->
+      </geometry>
+      <!-- Fin de la geometría. -->
+    </collision>
+    <!-- Fin del bloque 'collision'. -->
+  </link>
+  <!-- Fin de la definición del enlace. -->
   <joint name="joint_4" type="revolute">
+  <!-- Articulación 'joint_4' de tipo 'revolute' que conecta dos enlaces. -->
     <parent link="claw_support" />
+    <!-- Especifica el enlace padre conectado por esta articulación. -->
     <child link="gripper_right" />
+    <!-- Especifica el enlace hijo conectado por esta articulación. -->
     <origin xyz="-0.04 0.13 -0.1" rpy="0 0 0" />
+    <!-- Transformación del elemento: posición (xyz en m) y orientación (rpy en rad) respecto al marco padre. -->
     <axis xyz="0 0 1" />
+    <!-- Eje de movimiento de la articulación (vector unitario). -->
     <limit lower="-${PI/2}" upper="0.0" effort="${effort}" velocity="${velocity}" />
-  </joint>
+    <!-- Límites de la articulación: rango, esfuerzo y velocidad máximos. -->
+  </joint>
+  <!-- Fin de la articulación. -->
   <joint name="joint_5" type="revolute">
+  <!-- Articulación 'joint_5' de tipo 'revolute' que conecta dos enlaces. -->
     <parent link="claw_support" />
+    <!-- Especifica el enlace padre conectado por esta articulación. -->
     <child link="gripper_left" />
+    <!-- Especifica el enlace hijo conectado por esta articulación. -->
     <origin xyz="-0.22 0.13 -0.1" rpy="0 0 0" />
+    <!-- Transformación del elemento: posición (xyz en m) y orientación (rpy en rad) respecto al marco padre. -->
     <axis xyz="0 0 1" />
+    <!-- Eje de movimiento de la articulación (vector unitario). -->
     <mimic joint="joint_4" multiplier="-1"/>
     <limit lower="0.0" upper="${PI/2}" effort="${effort}" velocity="${velocity}" />
-  </joint>
+    <!-- Límites de la articulación: rango, esfuerzo y velocidad máximos. -->
+  </joint>
+  <!-- Fin de la articulación. -->
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
Commit message: ya casi acabo

File: arduinobot_ws/src/arduinobot_description/urdf/arduinobot.urdf.xacro (robot description, xacro)
@@ -3,4 +3,5 @@
 <robot xmlns:xacro="http://www.ros.org/wiki/xacro" name="arduinobot">
 <!-- Elemento raíz URDF; define el nombre del robot y el espacio de nombres de Xacro. -->
+  <xacro:arg name="is_sim" default="true"/>
   <xacro:arg name="is_ignition" default="true"/>
   <xacro:include filename="$(find arduinobot_description)/urdf/arduinobot_gazebo.xacro" />

File: arduinobot_ws/src/arduinobot_description/urdf/arduinobot_ros2_control.xacro (robot description, xacro)
@@ -2,4 +2,24 @@
 <robot xmlns:xacro="http://www.ros.org/wiki/xacro" name="arduinobot">
     <ros2_control name="RobotSystem" type="system">
+        <xacro:if value="$(arg is_sim)">
+            <hardware>
+                <plugin>gazebo_ros2_control/GazeboSystem</plugin>
+            </hardware>
+            <!-- lO SIGUIENTE ES SOLO PARA LA SIMULACION-->
+            <joint name="joint_5">
+                <param name="mimic">joint_4</param>
+                <param name="multiplier">-1</param>
+                <command_interface name="position">
+                    <param name="min">0.0</param>
+                    <param name="max">${PI / 2}</param>
+                </command_interface>
+            </joint>
+        </xacro:if>
+        <xacro:unless value="$(arg is_sim)">
+            <hardware>
+                <plugin>arduinobot_controller/ArduinobotInterface</plugin>
+                <param nmae="port">/dev/ttyUSB0</param>
+            </hardware>
+        </xacro:unless>
         <xacro:property name="PI" value="3.14159265359" />
         <!-- ros2_control Gazebo -->
@@ -18,6 +38,6 @@
         <joint name="joint_1">
             <command_interface name="position">
-            <param name="min">-${PI / 2}</param>
-            <param name="max">${PI / 2}</param>
+                <param name="min">-${PI / 2}</param>
+                <param name="max">${PI / 2}</param>
             </command_interface>
             <state_interface name="position"/>
@@ -25,6 +45,6 @@
         <joint name="joint_2">
             <command_interface name="position">
-            <param name="min">-${PI / 2}</param>
-            <param name="max">${PI / 2}</param>
+                <param name="min">-${PI / 2}</param>
+                <param name="max">${PI / 2}</param>
             </command_interface>
             <state_interface name="position"/>
@@ -32,6 +52,6 @@
         <joint name="joint_3">
             <command_interface name="position">
-            <param name="min">-${PI / 2}</param>
-            <param name="max">${PI / 2}</param>
+                <param name="min">-${PI / 2}</param>
+                <param name="max">${PI / 2}</param>
             </command_interface>
             <state_interface name="position"/>
@@ -39,13 +59,9 @@
         <joint name="joint_4">
             <command_interface name="position">
-            <param name="min">-${PI / 2}</param>
-            <param name="max">0.0</param>
+                <param name="min">-${PI / 2}</param>
+                <param name="max">0.0</param>
             </command_interface>
             <state_interface name="position"/>
         </joint>
-        <joint name="joint_5">
-            <param name="mimic">joint_4</param>
-            <param name="multiplier">-1</param>
-        </joint>
     </ros2_control>
 </robot>
