Commit message: poco, falta poco

File: arduinobot_ws/src/arduinobot_description/urdf/arduinobot_ros2_control.xacro (robot description, xacro)
@@ -1,4 +1,5 @@
 <?xml version="1.0"?>
 <robot xmlns:xacro="http://www.ros.org/wiki/xacro" name="arduinobot">
+    <xacro:property name="PI" value="3.14159265359" />
     <ros2_control name="RobotSystem" type="system">
         <xacro:if value="$(arg is_sim)">
@@ -22,5 +23,4 @@
             </hardware>
         </xacro:unless>
-        <xacro:property name="PI" value="3.14159265359" />
         <!-- ros2_control Gazebo -->
         <!-- ROS 2 Humble -->
